Commit message: Add control update

File: src/capbot_description/urdf/capbot.urdf (robot description, URDF)
Before this commit: robot capbot, 4 links, 3 joints
Links:
- link L_Link: mass 0.15555 -> 0.21431
- link R_Link: mass 0.15555 -> 0.21431
- link base_link: mass 3.4164 -> 8.127
- link laser: mass 1e-5 -> 0; geometry collision mesh filename=package://capbot_description/meshes/rplidar_Link.STL; visual mesh filename=package://capbot_description/meshes/rplidar_Link.STL
Joints:
- joint L_joint: axis 0 0 0 -> 0 0 1; origin xyz=0.244 0 0 rpy=1.5708 0 1.5708 -> xyz=0 0.238 0 rpy=1.5708 0 3.1416
- joint R_joint: axis 0 0 0 -> 0 0 1; origin xyz=-0.243 0 0 rpy=1.5708 0 1.5708 -> xyz=0 -0.238 0 rpy=1.5708 -1.1915 3.1415
- joint rplidar_joint: axis 0 1 0 -> 0 0 0; origin xyz=0 0 0.2 rpy=0 0 0 -> xyz=0.0 -0.0 0.2234 rpy=0 0 0
